Commit message: Add files via upload
二指夹爪初始版本

File: resources/qarm/urdf/QARM.urdf (robot description, URDF)
Before this commit: robot QARM, 6 links, 5 joints
Links:
- added link soft_gripper; visual mesh filename=../meshes/soft_gripper_visual.stl scale=1 1 1
Joints:
- added joint ee_to_soft_gripper: type fixed, parent END-EFFECTOR, child soft_gripper, origin xyz=0 0 0 rpy=0 0 0

Commit message: Add files via upload
qarm文件其实可选择修改（只影响打开时候的Figure1小图，不重要）

File: resources/qarm/urdf/QARM.urdf (robot description, URDF)
Before this commit: robot QARM, 6 links, 5 joints
Links:
- added link quad_fruit_gripper, mass 0.06; collision mesh filename=package://meshes/QARM_quad_fruit_gripper.stl scale=0.001 0.001 0.001; visual mesh filename=package://meshes/QARM_quad_fruit_gripper.stl scale=0.001 0.001 0.001
Joints:
- added joint ee_to_quad_fruit_gripper: type fixed, parent END-EFFECTOR, child quad_fruit_gripper, origin xyz=0 0 0.03 rpy=1.57079632679 0 0
